File: hhkb.kicad_pcb (KiCad board)
At the start: 2 copper layers, 285.8 x 98.6 mm, 136 parts, among them J1 USB_mini_micro_B, SW1 SW_PUSH, U1 ATMEGA32U4, X1 XTAL_GND

Commit message: rotate 90 degree
Parts:
- moved D6:12 268.6 mm to (36.5, 29.2), turned to 0 degrees
- moved D2:1 268.4 mm to (37.7, 302.9), turned to 0 degrees
- moved ESC1 263.1 mm to (39.8, 299.7), turned to 270 degrees
- moved D1:1 262.3 mm to (36.8, 295.9), turned to 0 degrees
- moved "`"1 261.5 mm to (39.8, 33.0), turned to 270 degrees
- moved D3:1 256.7 mm to (38.8, 292.3), turned to 0 degrees
- moved D7:12 255.5 mm to (37.5, 41.4), turned to 0 degrees
- moved D3:2 253.4 mm to (38.8, 288.9), turned to 0 degrees
- moved D2:2 251.3 mm to (37.8, 285.7), turned to 0 degrees
- moved D8:12 250.6 mm to (38.5, 45.4), turned to 0 degrees
- moved D:6:11 250.1 mm to (36.4, 48.2), turned to 0 degrees
- moved J1 244.8 mm to (30.3, 61.6), turned to 90 degrees
- moved "1"1 244.4 mm to (39.8, 280.7), turned to 270 degrees
- moved D1:2 244.1 mm to (36.8, 276.8), turned to 0 degrees
- moved "\"1 242.9 mm to (39.8, 52.1), turned to 270 degrees
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Other:
- board size 285.8 x 98.6 mm -> 98.6 x 285.8 mm

Commit message: change usb connector footprint
Parts:
- J1: footprint keyboard_parts:USB_miniB_hirose_5ST_hand -> keyboard_parts:USB_miniB_hirose_5S8
- moved D2:6 26.2 mm to (37.8, 181.6)
- moved D3:4 0.51 mm to (38.8, 249.8)
- moved D3:3 0.31 mm to (38.8, 268.6)
- moved D1:1 0.29 mm to (36.8, 296.2)
- moved D1:3 0.20 mm to (36.8, 258.0)
Routing:
- net Net-("6"1-Pad2): track 31.6 -> 2.57 mm
- net /ROW3: track 224.2 -> 218.5 mm
- net Net-(D10:11-Pad2): track 45.2 -> 50.4 mm
- net /ROW1: track 224.3 -> 228.1 mm
- net Net-(U1-Pad19): track 0.00 -> 3.40 mm
- net /ROW2: track 229.5 -> 232.8 mm
- net GND: track 914.0 -> 916.3 mm
- net Net-(U1-Pad18): track 0.00 -> 2.00 mm
- net Net-(D8:12-Pad2): track 36.6 -> 38.6 mm
- net Net-("O"1-Pad2): track 39.2 -> 41.0 mm
- net /COL12: track 192.3 -> 191.2 mm
- net Net-("]"1-Pad2): track 20.3 -> 20.8 mm
- net Net-(D9:11-Pad2): track 35.4 -> 36.0 mm
- added copper zone on B.Cu, net Net-(J1-Pad6)
Other:
- board size 98.6 x 285.8 mm -> 101.9 x 285.8 mm
