File: hhkb.kicad_pcb (KiCad board)
At the start: 2 copper layers, 101.2 x 276.2 mm, 140 parts, among them J1 USB_mini_micro_B, SW1 SW_PUSH, U1 ATMEGA32U4, X1 XTAL_GND

Commit message: optimize path
Routing:
- net /ROW9: track 321.5 -> 346.6 mm
- net /COL9: track 279.8 -> 291.2 mm
- net /COL10: track 327.6 -> 338.0 mm, vias 6 -> 5
- net /ROW10: track 274.3 -> 280.7 mm

Commit message: Rework from scratch
Parts:
- removed D10:10, D10:11, D10:12, D10:7, D10:8, D10:9, D5:1, D5:4, D5:5, D6:12, D6:7, D6:8, D6:9, D7:10, D7:11, D7:12, D7:8, D7:9, D8:10, D8:11, D8:12, D8:7, D8:8, D8:9, D9:10, D9:11, D9:12, D9:7, D9:8, D9:9, D:6:10, D:6:11, D:7:7: D, Diodes_THT:D_T-1_P12.70mm_Horizontal
- removed HOLE_M3 (x6): VAL**, keyboard_parts:HOLE_M3
- added D1:1: D, Diodes_THT:D_T-1_P10.16mm_Horizontal, F.Cu at (67.0, 348.1)
- added D1:10: D, Diodes_THT:D_T-1_P12.70mm_Horizontal, F.Cu at (67.2, 171.0)
- added D1:11: D, Diodes_THT:D_T-1_P12.70mm_Horizontal, F.Cu at (67.2, 151.9)
- added D1:12: D, Diodes_THT:D_T-1_P12.70mm_Horizontal, F.Cu at (67.2, 132.9)
- added D1:13: D, Diodes_THT:D_T-1_P12.70mm_Horizontal, F.Cu at (69.6, 113.8)
- added D1:14: D, Diodes_THT:D_T-1_P12.70mm_Horizontal, F.Cu at (67.3, 109.7)
- added D1:7: D, Diodes_THT:D_T-1_P12.70mm_Horizontal, F.Cu at (67.2, 228.1)
- added D1:8: D, Diodes_THT:D_T-1_P12.70mm_Horizontal, F.Cu at (67.2, 209.1)
- added D1:9: D, Diodes_THT:D_T-1_P12.70mm_Horizontal, F.Cu at (67.2, 190.0)
- added D2:10: D, Diodes_THT:D_T-1_P12.70mm_Horizontal, F.Cu at (86.2, 180.5)
- added D2:11: D, Diodes_THT:D_T-1_P12.70mm_Horizontal, F.Cu at (86.2, 161.5)
- added D2:12: D, Diodes_THT:D_T-1_P12.70mm_Horizontal, F.Cu at (86.2, 142.4)
- added D2:13: D, Diodes_THT:D_T-1_P12.70mm_Horizontal, F.Cu at (86.2, 123.4)
- added D2:14: D, Diodes_THT:D_T-1_P12.70mm_Horizontal, F.Cu at (67.3, 129.8)
- added D2:7: D, Diodes_THT:D_T-1_P12.70mm_Horizontal, F.Cu at (86.2, 237.7)
- added D2:8: D, Diodes_THT:D_T-1_P12.70mm_Horizontal, F.Cu at (86.2, 218.6)
- added D2:9: D, Diodes_THT:D_T-1_P12.70mm_Horizontal, F.Cu at (86.2, 199.6)
- added D3:10: D, Diodes_THT:D_T-1_P12.70mm_Horizontal, F.Cu at (105.3, 175.8)
- added D3:11: D, Diodes_THT:D_T-1_P12.70mm_Horizontal, F.Cu at (105.3, 156.7)
- added D3:12: D, Diodes_THT:D_T-1_P12.70mm_Horizontal, F.Cu at (105.3, 137.7)
- added D3:13: D, Diodes_THT:D_T-1_P12.70mm_Horizontal, F.Cu at (105.3, 113.8)
- added D3:7: D, Diodes_THT:D_T-1_P12.70mm_Horizontal, F.Cu at (105.3, 232.9)
- added D3:8: D, Diodes_THT:D_T-1_P12.70mm_Horizontal, F.Cu at (105.3, 213.9)
- added D3:9: D, Diodes_THT:D_T-1_P12.70mm_Horizontal, F.Cu at (105.3, 194.8)
- added D4:10: D, Diodes_THT:D_T-1_P12.70mm_Horizontal, F.Cu at (124.3, 166.2)
- added D4:11: D, Diodes_THT:D_T-1_P12.70mm_Horizontal, F.Cu at (124.3, 147.2)
- added D4:12: D, Diodes_THT:D_T-1_P12.70mm_Horizontal, F.Cu at (108.8, 123.4)
- added D4:13: D, Diodes_THT:D_T-1_P12.70mm_Horizontal, F.Cu at (108.8, 118.6)
- added D4:7: D, Diodes_THT:D_T-1_P12.70mm_Horizontal, F.Cu at (124.3, 223.4)
- added D4:8: D, Diodes_THT:D_T-1_P12.70mm_Horizontal, F.Cu at (124.3, 204.3)
- added D4:9: D, Diodes_THT:D_T-1_P12.70mm_Horizontal, F.Cu at (124.3, 185.3)
- added D5:10: D, Diodes_THT:D_T-1_P12.70mm_Horizontal, F.Cu at (126.7, 166.2)
- added D5:11: D, Diodes_THT:D_T-1_P12.70mm_Horizontal, F.Cu at (126.7, 147.2)
- added REF**: MountingHole_3mm_Pad, Mounting_Holes:MountingHole_3mm_Pad, F.Cu at (116.0, 363.9)
- added REF**: MountingHole_3mm_Pad, Mounting_Holes:MountingHole_3mm_Pad, F.Cu at (135.0, 304.3)
- added REF**: MountingHole_3mm_Pad, Mounting_Holes:MountingHole_3mm_Pad, F.Cu at (135.0, 190.0)
- added REF**: MountingHole_3mm_Pad, Mounting_Holes:MountingHole_3mm_Pad, F.Cu at (77.9, 97.2)
- added REF**: MountingHole_3mm_Pad, Mounting_Holes:MountingHole_3mm_Pad, F.Cu at (68.4, 294.8)
- added REF**: MountingHole_3mm_Pad, Mounting_Holes:MountingHole_3mm_Pad, F.Cu at (87.4, 206.7)
- D1:2: footprint Diodes_THT:D_T-1_P10.16mm_Horizontal -> Diodes_THT:D_T-1_P12.70mm_Horizontal
- moved D1:2 56.0 mm to (69.6, 299.6)
- moved D4:6 37.0 mm to (124.3, 242.4)
- moved C5 27.0 mm to (55.4, 326.4), turned to 180 degrees
- moved D1:4 26.2 mm to (67.2, 285.3)
- moved D1:5 26.2 mm to (67.2, 266.2)
- moved D1:6 26.2 mm to (67.2, 247.2)
- moved D5:2 24.1 mm to (124.3, 327.0), turned to 270 degrees
- moved D5:3 24.1 mm to (124.3, 303.2), turned to 270 degrees
- moved D3:6 21.5 mm to (105.3, 252.0)
- moved D5:6 18.2 mm to (126.7, 231.7), turned to 270 degrees
- moved D2:6 18.0 mm to (86.2, 256.7)
- moved D4:5 18.0 mm to (124.3, 261.5)
- moved D4:1 16.7 mm to (124.3, 342.4)
- moved D4:2 12.0 mm to (124.3, 318.6)
- moved D4:3 12.0 mm to (124.3, 299.6)
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Connections:
- "'"1 pad 1: /COL11 -> /ROW3
- ","1 pad 1: /COL10 -> /ROW4
- "-"1 pad 1: /COL9 -> /ROW1
- "."1 pad 1: /COL9 -> /ROW4
- "/"1 pad 1: /COL10 -> /ROW4
- "0"1 pad 1: /COL8 -> /ROW1
- "1"1 pad 1: /COL2 -> /ROW1
- "2"1 pad 1: /COL3 -> /ROW1
- "3"1 pad 1: /COL4 -> /ROW1
- "4"1 pad 1: /COL5 -> /ROW1
- "5"1 pad 1: /COL6 -> /ROW1
- "6"1 pad 1: /COL6 -> /ROW1
- "7"1 pad 1: /COL7 -> /ROW1
- "8"1 pad 1: /COL7 -> /ROW1
- "9"1 pad 1: /COL7 -> /ROW1
- ";"1 pad 1: /COL10 -> /ROW3
- "="1 pad 1: /COL10 -> /ROW1
- "A"1 pad 1: /COL2 -> /ROW3
- "B"1 pad 1: /COL4 -> /ROW4
- "C"1 pad 1: /COL3 -> /ROW4
- "D"1 pad 1: /COL4 -> /ROW3
- "E"1 pad 1: /COL4 -> /ROW2
- "F"1 pad 1: /COL5 -> /ROW3
- "G"1 pad 1: /COL5 -> /ROW3
- "H"1 pad 1: /COL5 -> /ROW3
- "I"1 pad 1: /COL8 -> /ROW2
- "J"1 pad 1: /COL7 -> /ROW3
- "K"1 pad 1: /COL8 -> /ROW3
- "L"1 pad 1: /COL9 -> /ROW3
- "M"1 pad 1: /COL9 -> /ROW4
- "N"1 pad 1: /COL8 -> /ROW4
- "O"1 pad 1: /COL8 -> /ROW2
- "P"1 pad 1: /COL9 -> /ROW2
- "Q"1 pad 1: /COL2 -> /ROW2
- "R"1 pad 1: /COL5 -> /ROW2
- "S"1 pad 1: /COL3 -> /ROW3
- "T"1 pad 1: /COL6 -> /ROW2
- "U"1 pad 1: /COL7 -> /ROW2
- "V"1 pad 1: /COL4 -> /ROW4
- "W"1 pad 1: /COL3 -> /ROW2
- "X"1 pad 1: /COL2 -> /ROW4
- "Y"1 pad 1: /COL6 -> /ROW2
- "Z"1 pad 1: /COL1 -> /ROW4
- "["1 pad 1: /COL10 -> /ROW2
- "\"1 pad 1: /COL11 -> /ROW1
- "]"1 pad 1: /COL11 -> /ROW2
- "`"1 pad 1: /COL12 -> /ROW1
- ALT1 pad 1: /COL2 -> /ROW5
- BS1 pad 1: /COL12 -> /ROW2
- CTRL1 pad 1: /COL1 -> /ROW3
- D1:2 pad 1: /ROW1 -> /COL2
- D1:2 pad 2: Net-("1"1-Pad2) -> Net-("2"1-Pad2)
- D1:3 pad 1: /ROW1 -> /COL3
- D1:3 pad 2: Net-("2"1-Pad2) -> Net-("3"1-Pad2)
- D1:4 pad 1: /ROW1 -> /COL4
- D1:4 pad 2: Net-("3"1-Pad2) -> Net-("4"1-Pad2)
- D1:5 pad 1: /ROW1 -> /COL5
- D1:5 pad 2: Net-("4"1-Pad2) -> Net-("5"1-Pad2)
- D1:6 pad 1: /ROW1 -> /COL6
- D1:6 pad 2: Net-("5"1-Pad2) -> Net-("6"1-Pad2)
- D2:1 pad 1: /ROW2 -> /COL1
- D2:2 pad 1: /ROW2 -> /COL2
- D2:3 pad 1: /ROW2 -> /COL3
- D2:4 pad 1: /ROW2 -> /COL4
- D2:5 pad 1: /ROW2 -> /COL5
- D2:6 pad 1: /ROW2 -> /COL6
- D2:6 pad 2: Net-("6"1-Pad2) -> Net-("T"1-Pad2)
- D3:1 pad 1: /ROW3 -> /COL1
- D3:2 pad 1: /ROW3 -> /COL2
- D3:3 pad 1: /ROW3 -> /COL3
- D3:4 pad 1: /ROW3 -> /COL4
- D3:5 pad 1: /ROW3 -> /COL5
- D3:6 pad 1: /ROW3 -> /COL6
- D3:6 pad 2: Net-("T"1-Pad2) -> Net-("G"1-Pad2)
- D4:1 pad 1: /ROW4 -> /COL1
- D4:1 pad 2: Net-("Z"1-Pad2) -> Net-(D4:1-Pad2)
- D4:2 pad 1: /ROW4 -> /COL2
- D4:2 pad 2: Net-("X"1-Pad2) -> Net-("Z"1-Pad2)
- D4:3 pad 1: /ROW4 -> /COL3
- D4:3 pad 2: Net-("C"1-Pad2) -> Net-("X"1-Pad2)
- D4:4 pad 1: /ROW4 -> /COL4
- D4:4 pad 2: Net-("V"1-Pad2) -> Net-("C"1-Pad2)
- D4:5 pad 1: /ROW4 -> /COL5
- D4:5 pad 2: Net-("G"1-Pad2) -> Net-("V"1-Pad2)
- D4:6 pad 1: /ROW4 -> /COL6
- D4:6 pad 2: Net-("Y"1-Pad2) -> Net-("B"1-Pad2)
- D5:2 pad 1: /ROW5 -> /COL2
- D5:3 pad 1: /ROW5 -> /COL3
- D5:6 pad 1: /ROW5 -> /COL6
- L_CMD1 pad 1: /COL3 -> /ROW5
- L_SHIFT1 pad 1: /COL1 -> /ROW4
- L_SHIFT1 pad 2: Net-(D5:1-Pad2) -> Net-(D4:1-Pad2)
- RET1 pad 1: /COL12 -> /ROW3
- R_ALT1 pad 1: /COL12 -> /ROW5
- R_CMD1 pad 1: /COL11 -> /ROW5
- R_FN1 pad 1: /COL12 -> /ROW4
- R_SHIFT1 pad 1: /COL11 -> /ROW4
- SPACEBAR1 pad 1: /COL6 -> /ROW5
- TAB1 pad 1: /COL1 -> /ROW2
- U1 pad 10: /COL3 -> (no net)
- U1 pad 11: /COL7 -> (no net)
- U1 pad 12: /COL6 -> /ROW1
- U1 pad 18: /COL5 -> /COL14
- U1 pad 19: /ROW6 -> /COL13
- U1 pad 20: /ROW7 -> /COL12
- U1 pad 21: /ROW8 -> /COL11
- U1 pad 22: /ROW1 -> /COL10
- U1 pad 25: /COL11 -> /COL9
- U1 pad 27: /ROW9 -> /COL3
- U1 pad 28: /ROW10 -> /COL6
- U1 pad 29: /COL10 -> /COL5
- U1 pad 30: /COL9 -> (no net)
- U1 pad 31: /COL4 -> /ROW2
- U1 pad 32: /ROW2 -> /COL4
- U1 pad 36: (no net) -> /COL7
- U1 pad 37: /ROW4 -> /ROW3
- U1 pad 38: /ROW3 -> /ROW4
- U1 pad 39: /ROW5 -> /COL2
- U1 pad 40: /COL1 -> /ROW5
- U1 pad 41: /COL2 -> /COL1
- U1 pad 8: /COL12 -> (no net)
Routing:
- net /ROW9: track 346.6 -> 0.00 mm, vias 1 -> 0
- net /COL13: track 0.00 -> 281.6 mm
- net /ROW10: track 280.7 -> 0.00 mm, vias 1 -> 0
- net /ROW6: track 264.1 -> 0.00 mm, vias 1 -> 0
- net /ROW8: track 262.6 -> 0.00 mm, vias 4 -> 0
- net /ROW7: track 233.8 -> 0.00 mm, vias 3 -> 0
- net /COL14: track 0.00 -> 227.8 mm
- net /ROW1: track 115.2 -> 309.4 mm, vias 4 -> 2
- net /ROW2: track 146.5 -> 313.1 mm
- net /COL11: track 394.5 -> 251.2 mm, vias 5 -> 0
- net /ROW4: track 192.2 -> 329.5 mm, vias 1 -> 2
- net /ROW3: track 169.9 -> 299.5 mm, vias 1 -> 2
- net /COL12: track 389.9 -> 261.0 mm
- net /COL10: track 338.0 -> 229.0 mm, vias 5 -> 0
- net /COL8: track 276.8 -> 192.3 mm, vias 2 -> 0
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
Commit message: redraw
Parts:
- D1:10, D1:11, D1:12, D1:2, D1:3, D1:4, D1:5, D1:8, D1:9, D2:1, D2:10, D2:11, D2:12, D2:13, D2:14, D2:2, D2:3, D2:4, D2:5, D2:6, D2:7, D2:8, D2:9, D3:1, D3:10, D3:11, D3:12, D3:13, D3:2, D3:3, D3:4, D3:5, D3:6, D3:7, D3:8, D3:9, D4:1, D4:10, D4:11, D4:12, D4:13, D4:2, D4:3, D4:4, D4:5, D4:6, D4:7, D4:8, D4:9, D5:10, D5:11, D5:2, D5:3, D5:6: footprint Diodes_THT:D_T-1_P12.70mm_Horizontal -> Diodes_THT:D_T-1_P10.16mm_Horizontal
- D1:13, D1:14, D1:6, D1:7: footprint Diodes_THT:D_T-1_P12.70mm_Horizontal -> Diodes_THT:D_T-1_P5.08mm_Horizontal
- J1: footprint keyboard_parts:USB_miniB_hirose_5S8 -> keyboard_parts:USB_miniB_hirose_5ST_hand
- moved J1 295.0 mm to (184.0, 80.0), turned to 0 degrees
- moved R3 289.2 mm to (182.4, 85.2), turned to 90 degrees
- moved R4 288.4 mm to (184.2, 85.2), turned to 90 degrees
- moved C8 287.1 mm to (187.0, 85.4), turned to 90 degrees
- moved C7 281.3 mm to (179.6, 88.4), turned to 180 degrees
- moved R1 278.6 mm to (201.6, 90.8), turned to 270 degrees
- moved C5 275.6 mm to (188.8, 85.3), turned to 90 degrees
- moved C1 270.7 mm to (198.7, 93.3), turned to 315 degrees
- moved C6 266.9 mm to (176.8, 101.1), turned to 90 degrees
- moved X1 265.8 mm to (196.2, 95.9), turned to 315 degrees
- moved C4 265.3 mm to (194.2, 90.7)
- moved SW1 265.1 mm to (209.8, 96.0), turned to 90 degrees
- moved U1 265.0 mm to (185.2, 96.2), turned to 270 degrees
- moved C2 262.5 mm to (199.3, 98.7), turned to 45 degrees
- moved "1"1 261.6 mm to (60.2, 90.3), turned to 0 degrees
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Connections:
- "-"1 pad 1: /ROW1 -> /ROW6
- "0"1 pad 1: /ROW1 -> /ROW6
- "8"1 pad 1: /ROW1 -> /ROW6
- "9"1 pad 1: /ROW1 -> /ROW6
- "="1 pad 1: /ROW1 -> /ROW6
- "\"1 pad 1: /ROW1 -> /ROW6
- "`"1 pad 1: /ROW1 -> /ROW3
- BS1 pad 1: /ROW2 -> /ROW4
- D1:14 pad 1: /COL14 -> /COL13
- D2:14 pad 1: /COL14 -> /COL13
- D3:13 pad 1: /COL13 -> /COL12
- RET1 pad 1: /ROW3 -> /ROW4
- R_FN1 pad 1: /ROW4 -> /ROW5
- R_SHIFT1 pad 1: /ROW4 -> /ROW5
- U1 pad 12: /ROW1 -> (no net)
- U1 pad 18: /COL14 -> /COL8
- U1 pad 26: /COL8 -> /ROW3
- U1 pad 27: /COL3 -> /ROW4
- U1 pad 28: /COL6 -> /ROW5
- U1 pad 29: /COL5 -> (no net)
- U1 pad 30: (no net) -> /ROW2
- U1 pad 31: /ROW2 -> /COL6
- U1 pad 32: /COL4 -> /COL5
- U1 pad 36: /COL7 -> /COL4
- U1 pad 37: /ROW3 -> /COL7
- U1 pad 38: /ROW4 -> /COL3
- U1 pad 40: /ROW5 -> /COL1
- U1 pad 41: /COL1 -> /ROW1
- U1 pad 8: (no net) -> /ROW6
Routing:
- net /COL14: track 227.8 -> 0.00 mm
- net /ROW1: track 309.4 -> 155.0 mm, vias 2 -> 0
- net /COL13: track 281.6 -> 155.4 mm
- net /ROW6: track 0.00 -> 116.2 mm
- net /COL1: track 74.8 -> 179.4 mm
- net /COL8: track 192.3 -> 88.9 mm
- net /COL9: track 210.6 -> 110.7 mm
- net /COL10: track 229.0 -> 129.2 mm
- net /COL7: track 178.7 -> 81.4 mm, vias 2 -> 0
- net GND: track 161.3 -> 255.5 mm, vias 6 -> 0
- net /COL12: track 261.0 -> 168.7 mm
- net /COL11: track 251.2 -> 159.0 mm
- net /ROW3: track 299.5 -> 377.6 mm, vias 2 -> 3
- net /COL3: track 98.0 -> 153.4 mm
- net /COL6: track 167.8 -> 126.6 mm
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- added copper zone on B.Cu, net GND
- added copper zone on F.Cu, net VCC
- removed copper zone on F.Cu, net GND
- removed copper zone on B.Cu, net VCC
Other:
- board size 101.2 x 276.2 mm -> 276.2 x 106 mm

Commit message: Change usb footprint
Parts:
- J1: footprint keyboard_parts:USB_miniB_hirose_5ST_hand -> keyboard_parts:USB_miniB_through_hole
Routing:
- net Net-(J1-Pad6): track 0.00 -> 24.1 mm
- net VCC: track 100.0 -> 81.3 mm, vias 1 -> 0
- net (no net): track 9.48 -> 0.00 mm
- net GND: track 255.5 -> 258.8 mm
- net Net-(J1-Pad2): track 4.18 -> 5.38 mm

Commit message: Gen gerbers
Parts:
- moved "`"1 283.2 mm to (32.7, 23.2), turned to 90 degrees
- moved REF** 279.3 mm to (51.8, 16.1), turned to 0 degrees
- moved D1:13 271.6 mm to (33.1, 32.7), turned to 180 degrees
- moved D1:14 265.1 mm to (41.4, 33.0), turned to 90 degrees
- moved BS1 264.2 mm to (51.8, 28.0), turned to 90 degrees
- moved "\"1 260.6 mm to (32.7, 42.3), turned to 90 degrees
- moved D2:14 249.2 mm to (57.3, 37.1), turned to 180 degrees
- moved D4:13 249.2 mm to (65.8, 33.1), turned to 0 degrees
- moved D1:12 244.9 mm to (38.5, 51.8), turned to 180 degrees
- moved R_FN1 244.4 mm to (89.9, 28.0), turned to 90 degrees
- moved D2:13 242.6 mm to (57.3, 42.3), turned to 180 degrees
- moved "="1 238.8 mm to (32.7, 61.3), turned to 90 degrees
- moved "]"1 234.7 mm to (51.8, 51.8), turned to 90 degrees
- moved RET1 234.4 mm to (70.8, 42.3), turned to 270 degrees
- moved D1:11 223.2 mm to (38.5, 70.9), turned to 180 degrees
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Routing:
- net GND: track 258.8 -> 810.7 mm
- net Net-(R2-Pad2): track 3.16 -> 6.22 mm
- net VCC: track 81.3 -> 82.8 mm
- net /ROW3: track 377.6 -> 378.9 mm
- net /ROW1: track 155.0 -> 153.8 mm
- net Net-("I"1-Pad2): track 16.5 -> 17.3 mm
Other:
- board size 276.2 x 106 mm -> 106 x 276.2 mm
